File: STM32F103C8T6/ST-Link/adaptor/adaptor.kicad_sch (KiCad schematic)
At the start: 4 parts, among them J1 Conn_01x20_Socket, J2 Conn_01x20_Socket, J3 Conn_01x04_Pin

Commit message: Place elements
Parts:
- R1: footprint Resistor_THT:R_Axial_DIN0207_L6.3mm_D2.5mm_P7.62mm_Horizontal -> Resistor_THT:R_Axial_DIN0204_L3.6mm_D1.6mm_P5.08mm_Horizontal
Connections:
- net 3.3V: now also J3.4 (Pin_4); no longer J3.1 (Pin_1)
- net GND: now also J3.1 (Pin_1); no longer J3.4 (Pin_4)
Changed lines of the file:
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@@
   (no_connect (at 158.75 83.185))
   (no_connect (at 186.69 37.465))
-  (wire (pts (xy 148.59 83.185) (xy 148.59 60.96))
+  (wire (pts (xy 148.59 60.96) (xy 148.59 83.185))
     (stroke (width 0) (type default))
   )
@@
     (stroke (width 0) (type default))
   )
-  (wire (pts (xy 207.645 41.275) (xy 207.645 63.5))
-    (stroke (width 0) (type default))
-  )
   (wire (pts (xy 146.05 66.675) (xy 151.13 66.675))
     (stroke (width 0) (type default))
   )
-  (wire (pts (xy 146.05 43.18) (xy 209.55 43.18))
+  (wire (pts (xy 146.05 43.18) (xy 201.295 43.18))
     (stroke (width 0) (type default))
   )
@@
     (stroke (width 0) (type default))
   )
-  (wire (pts (xy 209.55 43.18) (xy 209.55 55.88))
+  (wire (pts (xy 207.645 41.275) (xy 207.645 55.88))
+    (stroke (width 0) (type default))
+  )
+  (wire (pts (xy 201.295 43.18) (xy 201.295 63.5))
     (stroke (width 0) (type default))
   )
@@
     (stroke (width 0) (type default))
   )
-  (wire (pts (xy 209.55 55.88) (xy 217.17 55.88))
+  (wire (pts (xy 207.645 55.88) (xy 217.17 55.88))
     (stroke (width 0) (type default))
   )
-  (wire (pts (xy 151.13 66.675) (xy 151.13 58.42))
+  (wire (pts (xy 151.13 58.42) (xy 151.13 66.675))
     (stroke (width 0) (type default))
   )
@@
     (stroke (width 0) (type default))
   )
-  (wire (pts (xy 207.645 63.5) (xy 217.17 63.5))
+  (wire (pts (xy 201.295 63.5) (xy 217.17 63.5))
     (stroke (width 0) (type default))
   )
@@
     (effects (font (size 1.27 1.27)) (justify left bottom))
   )
-  (label "3.3V" (at 212.09 63.5 0) (fields_autoplaced)
+  (label "GND" (at 212.09 63.5 0) (fields_autoplaced)
+    (effects (font (size 0.8 0.8)) (justify left bottom))
+  )
+  (label "SWDIO" (at 212.09 58.42 0) (fields_autoplaced)
     (effects (font (size 0.8 0.8)) (justify left bottom))
   )
@@
     (effects (font (size 0.8 0.8)) (justify left bottom))
   )
-  (label "SWDIO" (at 212.09 58.42 0) (fields_autoplaced)
-    (effects (font (size 0.8 0.8)) (justify left bottom))
-  )
-  (label "GND" (at 212.09 55.88 0) (fields_autoplaced)
+  (label "3.3V" (at 212.09 55.88 0) (fields_autoplaced)
     (effects (font (size 0.8 0.8)) (justify left bottom))
   )
@@
       (effects (font (size 1.27 1.27)) (justify left))
     )
-    (property "Footprint" "Resistor_THT:R_Axial_DIN0207_L6.3mm_D2.5mm_P7.62mm_Horizontal" (at 144.272 74.93 90)
+    (property "Footprint" "Resistor_THT:R_Axial_DIN0204_L3.6mm_D1.6mm_P5.08mm_Horizontal" (at 144.272 74.93 90)
       (effects (font (size 1.27 1.27)) hide)
     )

Commit message: SWD socket connector
Parts:
- J3: footprint Connector_PinHeader_2.54mm:PinHeader_1x04_P2.54mm_Horizontal -> Connector_PinSocket_2.54mm:PinSocket_1x04_P2.54mm_Vertical
Changed lines of the file:
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@@
       (effects (font (size 1.27 1.27)) (justify right))
     )
-    (property "Footprint" "Connector_PinHeader_2.54mm:PinHeader_1x04_P2.54mm_Horizontal" (at 222.25 60.96 0)
+    (property "Footprint" "Connector_PinSocket_2.54mm:PinSocket_1x04_P2.54mm_Vertical" (at 222.25 60.96 0)
       (effects (font (size 1.27 1.27)) hide)
     )
